File: breakout/OV7670_breakout.kicad_pcb (KiCad board)
At the start: 2 copper layers, 25 x 43 mm, 5 parts, among them P101 CONN_02X10, P102 CONN_02X06, P103 CONN_02X06

Commit message: new breakout board
Parts:
- added C101: C, Capacitors_SMD:C_0805, F.Cu at (5.40, 17.6)
- added R103: R, Resistors_SMD:R_0805, F.Cu at (7.50, 29.5)
- added U101: DALC208, TO_SOT_Packages_SMD:SOT-23-6, F.Cu at (7.50, 19.5)
- moved R102 0.50 mm to (7.50, 34.5)
Connections:
- P101 pad 18: /JB4 -> Net-(P101-Pad18)
Routing:
- net /JA7: track 16.7 -> 54.8 mm, vias 0 -> 3
- net /JA1: track 16.0 -> 40.6 mm, vias 0 -> 3
- net /JB4: track 20.4 -> 7.19 mm
- net +3V3: track 51.6 -> 64.2 mm, vias 0 -> 3
- net Net-(P101-Pad18): track 0.00 -> 12.5 mm
- net /D6: track 19.8 -> 31.5 mm
- net /JB10: track 28.2 -> 21.0 mm, vias 0 -> 1
- net GND: track 0.00 -> 2.28 mm, vias 0 -> 2
- net /D7: track 19.1 -> 21.1 mm
- net /JB2: track 18.7 -> 19.7 mm
Other:
- rule pad_to_mask_clearance: 0.2 -> 0.06
- board text added: "Camera Breakout"
- board text added: "DO NOT PLUG IN WHEN FPGA IS POWERED"
- board text removed: "Camera Breakout wbraun@mit.edu"
