File: breakout/OV7670_breakout.sch (KiCad schematic (older format))
At the start: 5 parts, among them P101 CONN_02X10, P102 CONN_02X06, P103 CONN_02X06

Commit message: new breakout board
Parts:
- added C101: C, Capacitors_SMD:C_0805, symbol C
- added R103: R, Resistors_SMD:R_0805, symbol R
- added U101: DALC208, TO_SOT_Packages_SMD:SOT-23-6, symbol DALC208
Connections:
- net +3V3: now also C101.1, U101.2 (VCC)
- net GND: now also C101.2, U101.5 (VSS)
- net JA1: now also U101.3 (IO2)
- net JA7: now also U101.4 (IO3)
- net JB2: now also U101.1 (IO1)
- net JB4: now also R103.1; no longer P101.18 (P18)
- new net: P101.18 (P18), R103.2
Changed lines of the file:
@@
-EESchema Schematic File Version 2
+EESchema Schematic File Version 3
 LIBS:power
 LIBS:device
@@
 LIBS:contrib
 LIBS:valves
-EELAYER 25 0
+LIBS:wbraun_ic_lib
+LIBS:OV7670_breakout-cache
+EELAYER 26 0
 EELAYER END
 $Descr A4 11693 8268
@@
 	2900 5800 3000 5800
 Wire Wire Line
-	2900 5900 3000 5900
+	2900 5900 3300 5900
 Wire Wire Line
 	2400 5800 2300 5800
@@
 Text Label 2300 5200 2    60   ~ 0
 RST
-Text Label 3000 5900 0    60   ~ 0
+Text Label 3750 5900 0    60   ~ 0
 SIOD
 Text Label 3000 5800 0    60   ~ 0
@@
 Text Label 7300 4300 0    60   ~ 0
 SIOD
+$Comp
+L DALC208 U101
+U 1 1 59FCA1D9
+P 4700 1850
+F 0 "U101" H 4700 2287 60  0000 C CNN
+F 1 "DALC208" H 4700 2181 60  0000 C CNN
+F 2 "TO_SOT_Packages_SMD:SOT-23-6" H 4800 1250 60  0001 C CNN
+F 3 "" H 4800 1250 60  0001 C CNN
+	1    4700 1850
+	1    0    0    -1
+$EndComp
+Wire Wire Line
+	3900 1700 4250 1700
+Wire Wire Line
+	4150 1700 4150 1500
+Wire Wire Line
+	3900 2000 4250 2000
+Wire Wire Line
+	4150 2000 4150 2200
+$Comp
+L C C101
+U 1 1 59FCA4A3
+P 3900 1850
+F 0 "C101" H 4015 1896 50  0000 L CNN
+F 1 "C" H 4015 1805 50  0000 L CNN
+F 2 "Capacitors_SMD:C_0805" H 3938 1700 50  0001 C CNN
+F 3 "" H 3900 1850 50  0001 C CNN
+	1    3900 1850
+	1    0    0    -1
+$EndComp
+Connection ~ 4150 2000
+Connection ~ 4150 1700
+$Comp
+L +3V3 #PWR015
+U 1 1 59FCA74D
+P 4150 1500
+F 0 "#PWR015" H 4150 1350 50  0001 C CNN
+F 1 "+3V3" H 4150 1640 50  0000 C CNN
+F 2 "" H 4150 1500 50  0000 C CNN
+F 3 "" H 4150 1500 50  0000 C CNN
+	1    4150 1500
+	1    0    0    -1
+$EndComp
+$Comp
+L GND #PWR016
+U 1 1 59FCA7DD
+P 4150 2200
+F 0 "#PWR016" H 4150 1950 50  0001 C CNN
+F 1 "GND" H 4150 2050 50  0000 C CNN
+F 2 "" H 4150 2200 50  0000 C CNN
+F 3 "" H 4150 2200 50  0000 C CNN
+	1    4150 2200
+	1    0    0    -1
+$EndComp
+Wire Wire Line
+	5150 1700 5250 1700
+Wire Wire Line
+	5150 1800 5250 1800
+Wire Wire Line
+	5150 1900 5250 1900
+Wire Wire Line
+	5150 2000 5250 2000
+$Comp
+L R R103
+U 1 1 59FCA9D2
+P 3450 5900
+F 0 "R103" V 3530 5900 50  0000 C CNN
+F 1 "R" V 3450 5900 50  0000 C CNN
+F 2 "Resistors_SMD:R_0805" V 3380 5900 50  0001 C CNN
+F 3 "" H 3450 5900 50  0000 C CNN
+	1    3450 5900
+	0    1    1    0
+$EndComp
+Wire Wire Line
+	3600 5900 3750 5900
+Text Label 5250 1700 0    60   ~ 0
+XCLK
+Text Label 5250 1900 0    60   ~ 0
+RST
+Text Label 5250 1800 0    60   ~ 0
+PWDN
 $EndSCHEMATC

Commit message: updated kicad files
Parts:
- C101: symbol C -> OV7670_breakout-rescue:C
- P101: symbol CONN_02X10 -> OV7670_breakout-rescue:CONN_02X10
- P102, P103: symbol CONN_02X06 -> OV7670_breakout-rescue:CONN_02X06
- R101, R102, R103: symbol R -> OV7670_breakout-rescue:R
- U101: symbol DALC208 -> wbraun_lib:DALC208
Changed lines of the file:
@@
-EESchema Schematic File Version 3
-LIBS:power
-LIBS:device
-LIBS:transistors
-LIBS:conn
-LIBS:linear
-LIBS:regul
-LIBS:74xx
-LIBS:cmos4000
-LIBS:adc-dac
-LIBS:memory
-LIBS:xilinx
-LIBS:microcontrollers
-LIBS:dsp
-LIBS:microchip
-LIBS:analog_switches
-LIBS:motorola
-LIBS:texas
-LIBS:intel
-LIBS:audio
-LIBS:interface
-LIBS:digital-audio
-LIBS:philips
-LIBS:display
-LIBS:cypress
-LIBS:siliconi
-LIBS:opto
-LIBS:atmel
-LIBS:contrib
-LIBS:valves
-LIBS:wbraun_ic_lib
+EESchema Schematic File Version 4
 LIBS:OV7670_breakout-cache
 EELAYER 26 0
@@
 $EndDescr
 $Comp
-L CONN_02X10 P101
+L OV7670_breakout-rescue:CONN_02X10 P101
 U 1 1 57F3DEC6
 P 2650 5550
@@
 $EndComp
 $Comp
-L CONN_02X06 P102
+L OV7670_breakout-rescue:CONN_02X06 P102
 U 1 1 57F3DF59
 P 5250 4050
@@
 $EndComp
 $Comp
-L CONN_02X06 P103
+L OV7670_breakout-rescue:CONN_02X06 P103
 U 1 1 57F3DFC6
 P 5250 5050
@@
 $EndComp
 $Comp
-L GND #PWR01
+L power:GND #PWR01
 U 1 1 57F3E0D8
 P 5600 4200
@@
 $EndComp
 $Comp
-L GND #PWR02
+L power:GND #PWR02
 U 1 1 57F3E0F5
 P 4900 4200
@@
 $EndComp
 $Comp
-L GND #PWR03
+L power:GND #PWR03
 U 1 1 57F3E10F
 P 4900 5200
@@
 $EndComp
 $Comp
-L GND #PWR04
+L power:GND #PWR04
 U 1 1 57F3E129
 P 5600 5200
@@
 $EndComp
 $Comp
-L +3V3 #PWR05
+L power:+3V3 #PWR05
 U 1 1 57F3E161
 P 4900 5350
@@
 $EndComp
 $Comp
-L +3V3 #PWR06
+L power:+3V3 #PWR06
 U 1 1 57F3E17B
 P 5600 5350
@@
 $EndComp
 $Comp
-L +3V3 #PWR07
+L power:+3V3 #PWR07
 U 1 1 57F3E195
 P 4900 4350
@@
 $EndComp
 $Comp
-L +3V3 #PWR08
+L power:+3V3 #PWR08
 U 1 1 57F3E1AF
 P 5600 4350
@@
 PWDN
 $Comp
-L GND #PWR09
+L power:GND #PWR09
 U 1 1 57F3EA80
 P 3000 6000
@@
 $EndComp
 $Comp
-L GND #PWR010
+L power:GND #PWR010
 U 1 1 57F3EA9A
 P 2300 5100
@@
 	2200 2800 2400 2800
 $Comp
-L +3V3 #PWR011
+L power:+3V3 #PWR011
 U 1 1 57F3ED91
 P 2300 6000
@@
 $EndComp
 $Comp
-L GND #PWR012
+L power:GND #PWR012
 U 1 1 57F3EDAB
 P 3000 5100
@@
 JB4
 $Comp
-L R R101
+L OV7670_breakout-rescue:R R101
 U 1 1 57F3EFB6
 P 7100 3750
@@
 $EndComp
 $Comp
-L R R102
+L OV7670_breakout-rescue:R R102
 U 1 1 57F3F059
 P 7300 3750
@@
 $EndComp
 $Comp
-L +3V3 #PWR013
+L power:+3V3 #PWR013
 U 1 1 57F3F098
 P 7100 3500
@@
 $EndComp
 $Comp
-L +3V3 #PWR014
+L power:+3V3 #PWR014
 U 1 1 57F3F0B6
 P 7300 3500
@@
 SIOD
 $Comp
-L DALC208 U101
+L wbraun_lib:DALC208 U101
 U 1 1 59FCA1D9
 P 4700 1850
@@
 $EndComp
 Wire Wire Line
-	3900 1700 4250 1700
+	3900 1700 4150 1700
 Wire Wire Line
 	4150 1700 4150 1500
 Wire Wire Line
-	3900 2000 4250 2000
+	3900 2000 4150 2000
 Wire Wire Line
 	4150 2000 4150 2200
 $Comp
-L C C101
+L OV7670_breakout-rescue:C C101
 U 1 1 59FCA4A3
 P 3900 1850
@@
 Connection ~ 4150 1700
 $Comp
-L +3V3 #PWR015
+L power:+3V3 #PWR015
 U 1 1 59FCA74D
 P 4150 1500
@@
 $EndComp
 $Comp
-L GND #PWR016
+L power:GND #PWR016
 U 1 1 59FCA7DD
 P 4150 2200
@@
 	5150 2000 5250 2000
 $Comp
-L R R103
+L OV7670_breakout-rescue:R R103
 U 1 1 59FCA9D2
 P 3450 5900
@@
 Text Label 5250 1800 0    60   ~ 0
 PWDN
+Wire Wire Line
+	4150 2000 4250 2000
+Wire Wire Line
+	4150 1700 4250 1700
 $EndSCHEMATC
