File: breakout/camera_side_breakout/camera_side_breakout.kicad_pcb (KiCad board)
At the start: 2 copper layers, 18 x 28 mm, 2 parts, among them P101 CONN_02X09, P102 CONN_02X10

Commit message: new breakout board
Parts:
- added C101: C, Capacitors_SMD:C_0805, B.Cu at (120.7, 125.2)
- moved P102 1.50 mm to (126.5, 102.8)
Routing:
- net /3V3: track 10.7 -> 13.0 mm
- net /GND: track 10.6 -> 12.5 mm
- net /SIOC: track 10.6 -> 12.4 mm
- net /VSYNC: track 10.6 -> 12.1 mm
- net /RESET: track 10.6 -> 12.1 mm
- net /PCLK: track 10.6 -> 12.1 mm
- net /D7: track 10.6 -> 12.1 mm
- net /D5: track 10.6 -> 12.1 mm
- net /D3: track 10.6 -> 12.1 mm
- net /D1: track 10.6 -> 12.1 mm
- net /HREF: track 10.6 -> 12.1 mm
- net /XCLK: track 10.6 -> 12.1 mm
- net /SIOD: track 10.6 -> 12.1 mm
- net /PWDN: track 10.6 -> 12.1 mm
- net /D6: track 10.6 -> 12.1 mm
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Other:
- board size 18 x 28 mm -> 19.5 x 28 mm
- rule pad_to_mask_clearance: 0.1 -> 0.06
