File: breakout/camera_side_breakout/camera_side_breakout.sch (KiCad schematic (older format))
At the start: 2 parts, among them P101 CONN_02X09, P102 CONN_02X10

Commit message: new breakout board
Parts:
- added C101: C, Capacitors_SMD:C_0805, symbol C
Connections:
- net 3V3: now also C101.1
- net GND: now also C101.2
Changed lines of the file:
@@
-EESchema Schematic File Version 2
+EESchema Schematic File Version 3
 LIBS:power
 LIBS:device
@@
 LIBS:contrib
 LIBS:valves
-EELAYER 25 0
+LIBS:camera_side_breakout-cache
+EELAYER 26 0
 EELAYER END
 $Descr A4 11693 8268
@@
 Text Label 3800 4600 0    60   ~ 0
 SIOD
+$Comp
+L C C101
+U 1 1 59FCB06D
+P 4600 2550
+F 0 "C101" H 4715 2596 50  0000 L CNN
+F 1 "C" H 4715 2505 50  0000 L CNN
+F 2 "Capacitors_SMD:C_0805" H 4638 2400 50  0001 C CNN
+F 3 "" H 4600 2550 50  0001 C CNN
+	1    4600 2550
+	1    0    0    -1
+$EndComp
+Text Label 4600 2300 2    60   ~ 0
+3V3
+Text Label 4600 2800 0    60   ~ 0
+GND
+Wire Wire Line
+	4600 2300 4600 2400
+Wire Wire Line
+	4600 2700 4600 2800
 $EndSCHEMATC
